File: eagle/frankfurt_eth_pic.sch (EAGLE design)
At the start: 60 parts, among them IC1 PIC18F26K80, IC2 ENC28J60-SO, IC3 SN65HVD232, IC4 LM2575S, IC5 11AA02E48, IC6 MCP23A256, IC7 AT45DB041D, J2 A00-108-220-450, Q1 10 MHz, Q2 25 MHz

Commit message: Updated rev texts
Other:
- note added: "Frankfurt Eth"
- note added: "PIC version"
- note removed: "Ethernet"
- note removed: "Expansion"
- note removed: "Odessa"
- note removed: "http://www.grodansparadis.com"
Changed lines of the file:
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@@
 <text x="200.66" y="175.26" size="1.778" layer="91">Horizontal type</text>
 <text x="378.46" y="7.62" size="1.778" layer="91">A</text>
-<text x="289.56" y="27.94" size="5.08" layer="91">Odessa</text>
-<text x="365.76" y="25.4" size="1.778" layer="91">http://www.vscp.org</text>
-<text x="289.56" y="25.4" size="1.778" layer="91">Expansion</text>
 <text x="287.02" y="241.3" size="1.778" layer="91">Input voltage</text>
 <text x="287.02" y="238.76" size="1.778" layer="91">+7V DC - +28V DC</text>
@@
 <text x="127" y="66.04" size="1.778" layer="91">+3.3V</text>
 <text x="81.28" y="20.32" size="1.778" layer="91">+3.3V</text>
+<text x="289.56" y="27.94" size="5.08" layer="91">Frankfurt Eth</text>
+<text x="365.76" y="25.4" size="1.778" layer="91">http://www.vscp.org</text>
+<text x="289.56" y="25.4" size="1.778" layer="91">PIC version</text>
 </plain>
 <instances>
@@
 <sheet>
 <plain>
-<text x="292.1" y="17.78" size="1.778" layer="91">Ethernet</text>
 <text x="375.92" y="2.54" size="1.778" layer="91">Rev A</text>
-<text x="292.1" y="15.24" size="1.778" layer="91">http://www.grodansparadis.com</text>
+<text x="292.1" y="15.24" size="5.08" layer="91">Frankfurt Eth</text>
+<text x="292.1" y="7.62" size="1.778" layer="91">http://www.vscp.org</text>
+<text x="292.1" y="12.7" size="1.778" layer="91">PIC version</text>
 </plain>
 <instances>
@@
 <text x="99.06" y="162.56" size="1.778" layer="91">BUS WARNING</text>
 <text x="149.86" y="162.56" size="1.778" layer="91">BUS OFF</text>
+<text x="292.1" y="17.78" size="5.08" layer="91">Frankfurt Eth</text>
+<text x="292.1" y="10.16" size="1.778" layer="91">http://www.vscp.org</text>
+<text x="292.1" y="15.24" size="1.778" layer="91">PIC version</text>
+<text x="378.46" y="5.08" size="1.778" layer="91">A</text>
 </plain>
 <instances>
