File: pic-version/eagle/frankfurt_eth_pic.brd (EAGLE design)
At the start: 72.1 x 65.5 mm, 62 parts, among them IC1 PIC18F26K80, IC2 ENC28J60-SO, IC3 SN65HVD232, IC4 LM2575S, IC5 11AA02E48, IC6 MCP23A256, IC7 AT45DB041D, J2 A00-108-220-450, Q1 10 MHz, Q2 25 MHz

Commit message: Changed value of C14 to 10uF
Parts:
- C14: value 1 uF -> 10 uF
Changed lines of the file:
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@@
 </element>
 <element name="LED2" library="led" package="CHIP-LED0805" value="Red LED" x="51.45" y="18.8" smashed="yes" rot="R180"/>
-<element name="C14" library="rcl" package="C0805" value="1 uF" x="55.91" y="30.62" smashed="yes" rot="R180">
+<element name="C14" library="rcl" package="C0805" value="10 uF" x="55.91" y="30.62" smashed="yes" rot="R180">
 <attribute name="NAME" x="57.92" y="32.43" size="0.6096" layer="25" font="fixed" rot="R180"/>
 </element>
