File: esp32-version-poe/kicad/frakfurt_eth.kicad_pcb (KiCad board)
At the start: 2 copper layers, 42.1 x 72 mm, 43 parts, among them J1 HR911105A, J2 PROG, J4 Conn_Left_I2C, J5 Conn_01x02, U2 ESP32-WROOM-32, U3 LAN8720A, U4 SN65HVD232, U5 R-78B3.3-1.0 (Recom)

Commit message: Added gerbers
Parts:
- removed the REF** at (123.5, 78.2)
- added D5: GREEN, LED_SMD:LED_0805_2012Metric_Pad1.15x1.40mm_HandSolder, F.Cu at (110.7, 119.5)
- added D6: YELLO, LED_SMD:LED_0805_2012Metric_Pad1.15x1.40mm_HandSolder, F.Cu at (131.2, 119.2)
- added J3: Conn_01x02_Pin, Connector_PinHeader_2.54mm:PinHeader_1x02_P2.54mm_Vertical, F.Cu at (132.9, 106.8)
- added J6: Conn_01x02_Pin, Connector_PinHeader_2.54mm:PinHeader_1x02_P2.54mm_Vertical, F.Cu at (98.0, 81.7)
- added REF**: OSHW-Logo_5.7x6mm_SilkScreen, Symbol:OSHW-Logo_5.7x6mm_SilkScreen, F.Cu at (127.7, 76.0)
- J1: value HR911105A -> Taimag RJP-003TC1; footprint prjlocal:HANRUN_HR911105A -> Connector_RJ:RJ45_Abracon_ARJP11A-MA_Horizontal
- L1, L2: value BLM18PG181SN1D -> BLM21SP181SN1D
- moved J1 10.4 mm to (115.5, 106.7), turned to 0 degrees
- moved R14 3.60 mm to (132.1, 115.9), turned to 180 degrees
- moved R5 3.35 mm to (110.3, 116.2), turned to 180 degrees
Connections:
- J1 pad 10: Net-(J1-Pad10) -> /VIN-
- J1 pad 11: GND -> Net-(D5-A)
- J1 pad 12: Net-(J1-Pad12) -> GND
- J1 pad 15: GND -> unconnected-(J1-SHIELD-Pad15)
- J1 pad 4: +3V3 -> Net-(J1-CT-Pad4)
- J1 pad 5: +3V3 -> Net-(J1-CT-Pad4)
- J1 pad 7: (no net) -> GND
- J1 pad 9: +3V3 -> /VIN+
- L2 pad 1: Net-(J1-Pad4) -> Net-(J1-CT-Pad4)
- R1 pad 2: Net-(J1-Pad4) -> Net-(J1-CT-Pad4)
- R14 pad 2: Net-(J1-Pad12) -> Net-(D6-A)
- R2 pad 2: Net-(J1-Pad4) -> Net-(J1-CT-Pad4)
- R3 pad 2: Net-(J1-Pad4) -> Net-(J1-CT-Pad4)
- R4 pad 2: Net-(J1-Pad4) -> Net-(J1-CT-Pad4)
- R5 pad 2: Net-(J1-Pad10) -> Net-(D5-A)
Routing:
- net VBUS: track 3.47 -> 37.0 mm
- net Net-(J1-CT-Pad4): track 0.00 -> 29.7 mm, vias 0 -> 2
- net Net-(J1-Pad4): track 22.4 -> 0.00 mm, vias 2 -> 0
- net +3V3: track 294.1 -> 272.7 mm
- net GND: track 43.1 -> 53.3 mm
- net Net-(D5-A): track 0.00 -> 9.16 mm
- net Net-(D6-A): track 0.00 -> 8.92 mm
- net /VIN+: track 0.00 -> 8.28 mm
- net Net-(J1-Pad10): track 7.65 -> 0.00 mm
- net /VIN-: track 0.00 -> 7.01 mm
- net /RX+: track 17.7 -> 23.9 mm
- net /PHY_L2: track 40.4 -> 44.6 mm
- net Net-(J1-Pad12): track 4.19 -> 0.00 mm
- net /PHY_L1: track 35.3 -> 31.5 mm
- net /TX-: track 16.6 -> 19.9 mm
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Other:
- board text added: "Frankfurt Eth POE."
- board text removed: "Frankfurt Eth."
