File: esp32-version-poe/kicad/frakfurt_eth.kicad_sch (KiCad schematic)
At the start: 42 parts, among them J1 HR911105A, J2 PROG, J4 Conn_Left_I2C, J5 Conn_01x02, U2 ESP32-WROOM-32, U3 LAN8720A, U4 SN65HVD232, U5 R-78B3.3-1.0 (Recom)

Commit message: Added history file
Other:
- note added: "Connectors"
- note removed: "Misc"
Changed lines of the file:
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@@
     (effects (font (size 1.27 1.27)) (justify left bottom))
   )
-  (text "Misc" (at 12.7 101.6 0)
+  (text "Connectors" (at 12.7 101.6 0)
     (effects (font (size 1.27 1.27)) (justify left bottom))
   )

Commit message: Added gerbers
Parts:
- removed J1: HR911105A, lib:HANRUN_HR911105A, symbol HR911105A:HR911105A
- added D5: GREEN, LED_SMD:LED_0805_2012Metric_Pad1.15x1.40mm_HandSolder, symbol Device:LED
- added D6: YELLO, LED_SMD:LED_0805_2012Metric_Pad1.15x1.40mm_HandSolder, symbol Device:LED
- added J1: Taimag RJP-003TC1, Connector_RJ:RJ45_Abracon_ARJP11A-MA_Horizontal, symbol Connector:RJ45_Abracon_ARJP11A-MASA-B-A-EMU2
- added J3, J6: Conn_01x02_Pin, Connector_PinHeader_2.54mm:PinHeader_1x02_P2.54mm_Vertical, symbol Connector:Conn_01x02_Pin
- L1, L2: value BLM18PG181SN1D -> BLM21SP181SN1D
Connections:
- net GND: now also D5.1 (K), D6.1 (K), J1.12 (LLED-), J1.14 (RLED-), J1.7, J6.1 (Pin_1)
- net RX+: now also J1.3 (RD+)
- net RX-: now also J1.6 (RD-)
- net TX+: now also J1.1 (TD+)
- net TX-: now also J1.2 (TD-)
- net VBUS: now also J6.2 (Pin_2)
- net at L2.1, R1.2, R2.2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: now also J1.4 (CT), J1.5 (CT)
- net at R14.2: now also D6.2 (A), J1.13 (RLED+)
- net at R5.2: now also D5.2 (A), J1.11 (LLED+)
- new net VIN+: J1.9 (V+), J3.2 (Pin_2)
- new net VIN-: J1.10 (V-), J3.1 (Pin_1)
Other:
- moved on the sheet: L2, R1, R14, R2, R3, R4, R5
