File: esp32-version/kicad/frakfurt_eth.kicad_sch (KiCad schematic)
At the start: 42 parts, among them J1 HR911105A, J2 PROG, J4 Conn_Left_I2C, J5 Conn_01x02, U2 ESP32-WROOM-32, U3 LAN8720A, U4 SN65HVD232, U5 R-78B3.3-1.0 (Recom)

Commit message: Added gerbers
Parts:
- L1, L2: value BLM18PG181SN1D -> BLM21SP181SN1D
Changed lines of the file:
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@@
       (effects (font (size 1.27 1.27)))
     )
-    (property "Value" "BLM18PG181SN1D" (at 185.42 27.94 90)
+    (property "Value" "BLM21SP181SN1D" (at 185.42 27.94 90)
       (effects (font (size 1.27 1.27)))
     )
@@
       (effects (font (size 1.27 1.27)))
     )
-    (property "Value" "BLM18PG181SN1D" (at 50.8 106.68 90)
-      (effects (font (size 1.27 1.27)))
-    )
+    (property "Value" "BLM21SP181SN1D" (at 50.8 106.68 90)
+      (effects (font (size 1.27 1.27)))
+    )
