File: esp32-version/kicad/cpu.kicad_sch (KiCad schematic)
At the start: 10 parts, among them J2 PROG, U2 ESP32-WROOM-32

Commit message: Added som inital level II build code
Other:
- note added: "IMPORTANT"
- note added: "Later versions of ESP32 does not."
- note added: "ONLY ESP32-D0WD-V3 series have Ethernet MAC built in"
Changed lines of the file:
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@@
 		(comment 1 "http://www.vscp.org")
+	)
+	(text "Later versions of ESP32 does not."
+		(exclude_from_sim no)
+		(at 87.122 38.608 0)
+		(effects
+			(font
+				(size 1.27 1.27)
+			)
+		)
+	)
+	(text "ONLY ESP32-D0WD-V3 series have Ethernet MAC built in"
+		(exclude_from_sim no)
+		(at 98.298 35.814 0)
+		(effects
+			(font
+				(size 1.27 1.27)
+			)
+		)
+	)
+	(text "IMPORTANT"
+		(exclude_from_sim no)
+		(at 75.438 33.02 0)
+		(effects
+			(font
+				(size 1.27 1.27)
+			)
+		)
 	)
 	(text "Power"
