File: esp32-version/kicad/ethernet.kicad_sch (KiCad schematic)
At the start: 22 parts, among them J1 HR911105A, U3 LAN8720A

Commit message: Rearranged
Parts:
- J1: DESCRIPTION DIP RJ45 Connector; -> (none)
