File: esp32-version/kicad/frakfurt_eth.kicad_pcb (KiCad board)
At the start: 2 copper layers, 42.1 x 72 mm, 38 parts, among them J1 HR911105A, J2 PROG, J4 Conn_Left_I2C, J5 Conn_01x02, U2 ESP32-WROOM-32, U3 LAN8720A, U4 SN65HVD232, U5 R-78B3.3-1.0 (Recom)

Commit message: ESP32 version 1 preliminary done
Parts:
- removed the REF** at (123.6, 79.2)
- added D1: LED_Dual_KAK, LED_THT:LED_D5.0mm-3, F.Cu at (96.8, 61.1)
- added D4: LED, LED_SMD:LED_0805_2012Metric_Pad1.15x1.40mm_HandSolder, F.Cu at (100.5, 89.8)
- added L2: BLM18PG181SN1D, Resistor_SMD:R_0805_2012Metric_Pad1.20x1.40mm_HandSolder, F.Cu at (128.9, 103.3)
- added R16: 10k, Resistor_SMD:R_0805_2012Metric_Pad1.20x1.40mm_HandSolder, F.Cu at (99.3, 55.8)
- added R17: 470R, Resistor_SMD:R_0805_2012Metric_Pad1.20x1.40mm_HandSolder, F.Cu at (98.2, 89.8)
- added REF**: OSHW-Logo2_14.6x12mm_SilkScreen, Symbol:OSHW-Logo2_14.6x12mm_SilkScreen, F.Cu at (123.5, 78.2)
- C10, C11, C3, C6, C7, C8, C9: footprint Capacitor_SMD:C_0603_1608Metric -> Capacitor_SMD:C_0805_2012Metric_Pad1.18x1.45mm_HandSolder
- L1, R1, R10, R11, R12, R13, R14, R2, R3, R4, R5, R6, R7, R8, R9: footprint Resistor_SMD:R_0603_1608Metric -> Resistor_SMD:R_0805_2012Metric_Pad1.20x1.40mm_HandSolder
- moved C9 1.71 mm to (128.4, 88.6)
- moved R3 1.60 mm to (125.0, 103.3)
- moved C7 1.50 mm to (125.6, 88.5)
- moved R11 1.15 mm to (130.3, 98.5)
- moved R4 0.85 mm to (121.2, 103.3)
- moved R1 0.80 mm to (113.4, 103.3)
- moved R10 0.71 mm to (105.1, 67.5)
- moved R6 0.70 mm to (105.8, 56.8)
- moved C8 0.60 mm to (130.3, 96.3)
- moved J4 0.40 mm to (98.5, 119.0)
- moved R9 0.38 mm to (105.1, 65.5)
- moved R8 0.34 mm to (105.1, 63.5)
- moved R13 0.30 mm to (105.1, 61.3)
- moved C11 0.30 mm to (118.7, 94.5)
- moved C4 0.25 mm to (103.0, 53.8)
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Connections:
- net Net-(J4-Pin_2) renamed /CANH
- net Net-(J4-Pin_3) renamed /CANL
- R1 pad 2: +3V3 -> Net-(J1-Pad4)
- R2 pad 2: +3V3 -> Net-(J1-Pad4)
- R3 pad 2: +3V3 -> Net-(J1-Pad4)
- R4 pad 2: +3V3 -> Net-(J1-Pad4)
- U2 pad 6: unconnected-(U2-IO34-Pad6) -> /LEDA
- U2 pad 7: unconnected-(U2-IO35-Pad7) -> /LEDB
Routing:
- net Net-(J1-Pad4): track 0.00 -> 22.4 mm, vias 0 -> 2
- net /LEDA: track 0.00 -> 14.1 mm, vias 0 -> 1
- net +3V3: track 282.3 -> 294.1 mm
- net /PHY_L2: track 49.9 -> 40.4 mm
- net /LEDB: track 0.00 -> 7.67 mm, vias 0 -> 1
- net GND: track 36.4 -> 43.1 mm, vias 17 -> 36
- net Net-(D1-A): track 0.00 -> 5.17 mm
- net Net-(D4-A): track 0.00 -> 2.26 mm
- net Net-(U3-VDDCR): track 2.52 -> 4.09 mm
- net /RX+: track 19.0 -> 17.7 mm
- net /EN: track 30.1 -> 31.4 mm
- net Net-(U3-RXD1/MODE1): track 46.3 -> 45.1 mm
- net /PHY_L1: track 36.4 -> 35.3 mm, vias 2 -> 0
- net /RX-: track 13.1 -> 12.1 mm
- net Net-(U3-RXD0/MODE0): track 47.1 -> 48.1 mm
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- added copper zone on F.Cu, net GND
Other:
- board text added: "+3.3V"
- board text added: "BOOT0"
- board text added: "CANH"
- board text added: "CANL"
- board text added: "EN"
- board text added: "GND"
- board text added: "POWER"
- board text added: "RX"
- board text added: "STATUS"
- board text added: "TX"
- board text added: "Term."
- board text added: "VBUS"
